File: dsoxlan.kicad_pcb (KiCad board)
At the start: 2 copper layers, 81.3 x 58.4 mm, 14 parts, among them P1 7499010121A, P2 CONN_02X40

Commit message: Add the housing parts to schematics
This allows to assign them correct reference designators, and
removes the DRC warnings about schematic parity mismatches.
Parts:
- P1: footprint DSOXLAN:WURTH-7499010121A -> DSOXLAN:7499011121A
- moved P1 9.89 mm to (121.1, 88.3)
- renumbered REF** to N1, REF** to N2, REF** to N3
Connections:
- P1 pad 10: Net-(P1-AG) -> LED2
- P1 pad 11: LED2 -> Net-(P1-AG)
- P1 pad 12: Net-(P1-AY) -> LED1
- P1 pad 9: LED1 -> Net-(P1-AY)
- R1 pad 2: Net-(P1-AG) -> Net-(P1-AY)
- R2 pad 2: Net-(P1-AY) -> Net-(P1-AG)
Routing:
- net Net-(P1-AY): track 3.92 -> 39.3 mm
- net Net-(P1-AG): track 4.02 -> 27.4 mm
- net LED1: track 67.7 -> 90.0 mm
- net LED2: track 58.0 -> 79.1 mm
- net Net-(P1-CRD): track 16.3 -> 21.4 mm
- net TX+: track 64.9 -> 67.7 mm
- net TX-: track 64.9 -> 66.4 mm, vias 1 -> 2
- net RX-: track 69.4 -> 68.2 mm, vias 1 -> 2
- net +3.3V: track 87.3 -> 87.8 mm
- net GND: vias 31 -> 34
