File: dsoxlan.kicad_sch (KiCad schematic)
At the start: 11 parts, among them P1 7499010121A, P2 CONN_02X40

Commit message: Replace 7499010121A by 7499011121A
Parts:
- P1: footprint DSOXLAN:WURTH-7499010121A -> DSOXLAN:7499011121A; symbol dsoxlan:WÜRTH-7499010121A -> dsoxlan:WÜRTH-7499011121A
Connections:
- net LED1: now also P1.12 (KG); no longer P1.9 (KG)
- net LED2: now also P1.10 (KY); no longer P1.11 (KY)
- net at R2.2: now also P1.11 (AG); no longer P1.12 (AY)
- net at R1.2: now also P1.9 (AY); no longer P1.10 (AG)
Changed lines of the file:
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@@
+    (stroke (width 0) (type default))
+  )
+  (wire (pts (xy 90.17 104.14) (xy 95.25 104.14))
     (stroke (width 0) (type default))
   )
@@
     (stroke (width 0) (type default))
   )
+  (wire (pts (xy 90.17 96.52) (xy 95.25 96.52))
+    (stroke (width 0) (type default))
+  )
   (wire (pts (xy 80.01 76.2) (xy 80.01 83.82))
     (stroke (width 0) (type default))
@@
     (stroke (width 0) (type default))
   )
-  (wire (pts (xy 90.17 100.33) (xy 95.25 100.33))
-    (stroke (width 0) (type default))
-  )
   (wire (pts (xy 177.8 99.06) (xy 182.88 99.06))
     (stroke (width 0) (type default))
@@
   )
   (wire (pts (xy 170.18 99.06) (xy 170.18 101.6))
-    (stroke (width 0) (type default))
-  )
-  (wire (pts (xy 90.17 107.95) (xy 95.25 107.95))
     (stroke (width 0) (type default))
   )
@@
     )
   )
+  (global_label "LED1" (shape input) (at 82.55 107.95 0)
+    (effects (font (size 1.524 1.524)) (justify left))
+    (property "Intersheetrefs" "${INTERSHEET_REFS}" (at 82.55 107.95 0)
+      (effects (font (size 1.27 1.27)) hide)
+    )
+  )
   (global_label "RX+" (shape input) (at 180.34 104.14 180)
     (effects (font (size 1.524 1.524)) (justify right))
@@
     )
   )
+  (global_label "LED2" (shape input) (at 82.55 100.33 0)
+    (effects (font (size 1.524 1.524)) (justify left))
+    (property "Intersheetrefs" "${INTERSHEET_REFS}" (at 82.55 100.33 0)
+      (effects (font (size 1.27 1.27)) hide)
+    )
+  )
   (global_label "RX+" (shape input) (at 82.55 81.28 0)
     (effects (font (size 1.524 1.524)) (justify left))
@@
     )
   )
-  (global_label "LED1" (shape input) (at 82.55 96.52 0)
-    (effects (font (size 1.524 1.524)) (justify left))
-    (property "Intersheetrefs" "${INTERSHEET_REFS}" (at 82.55 96.52 0)
-      (effects (font (size 1.27 1.27)) hide)
-    )
-  )
   (global_label "TX+" (shape input) (at 180.34 93.98 180)
     (effects (font (size 1.524 1.524)) (justify right))
@@
     )
   )
-  (global_label "LED2" (shape input) (at 82.55 104.14 0)
-    (effects (font (size 1.524 1.524)) (justify left))
-    (property "Intersheetrefs" "${INTERSHEET_REFS}" (at 82.55 104.14 0)
-      (effects (font (size 1.27 1.27)) hide)
-    )
-  )
   (symbol (lib_id "power:GND") (at 67.31 116.84 0) (unit 1)
     (in_bom yes) (on_board yes) (dnp no)
@@
         (path "/071cacbe-efce-4cc8-8d6c-a55997c1e3c5"
           (reference "#PWR01") (unit 1)
-        )
-      )
-    )
-  )
-  (symbol (lib_id "Device:R") (at 86.36 107.95 270) (unit 1)
-    (in_bom yes) (on_board yes) (dnp no)
-    (property "Reference" "R2" (at 86.36 109.982 90)
-      (effects (font (size 1.016 1.016)))
-    )
-    (property "Value" "470R" (at 86.3854 108.1278 90)
-      (effects (font (size 1.016 1.016)))
-    )
-    (property "Footprint" "Resistor_SMD:R_0805_2012Metric_Pad1.20x1.40mm_HandSolder" (at 86.36 106.172 90)
-      (effects (font (size 1.27 1.27)) hide)
-    )
-    (property "Datasheet" "~" (at 86.36 107.95 0)
-      (effects (font (size 1.27 1.27)) hide)
-    )
-    (pin "1")
-    (pin "2")
-    (instances
-      (project "dsoxlan"
-        (path "/071cacbe-efce-4cc8-8d6c-a55997c1e3c5"
-          (reference "R2") (unit 1)
-        )
-      )
-    )
-  )
-  (symbol (lib_id "Device:R") (at 86.36 100.33 270) (unit 1)
-    (in_bom yes) (on_board yes) (dnp no)
-    (property "Reference" "R1" (at 86.36 102.362 90)
-      (effects (font (size 1.016 1.016)))
-    )
-    (property "Value" "470R" (at 86.3854 100.5078 90)
-      (effects (font (size 1.016 1.016)))
-    )
-    (property "Footprint" "Resistor_SMD:R_0805_2012Metric_Pad1.20x1.40mm_HandSolder" (at 86.36 98.552 90)
-      (effects (font (size 1.27 1.27)) hide)
-    )
-    (property "Datasheet" "~" (at 86.36 100.33 0)
-      (effects (font (size 1.27 1.27)) hide)
-    )
-    (pin "1")
-    (pin "2")
-    (instances
-      (project "dsoxlan"
-        (path "/071cacbe-efce-4cc8-8d6c-a55997c1e3c5"
-          (reference "R1") (unit 1)
-        )
-      )
-    )
-  )
-  (symbol (lib_id "power:+3.3V") (at 95.25 100.33 0) (unit 1)
-    (in_bom yes) (on_board yes) (dnp no)
-    (property "Reference" "#PWR02" (at 95.25 104.14 0)
-      (effects (font (size 1.524 1.524)) hide)
-    )
-    (property "Value" "+3V3" (at 95.25 96.774 0)
-      (effects (font (size 1.524 1.524)))
-    )
-    (property "Footprint" "" (at 95.25 100.33 0)
-      (effects (font (size 1.27 1.27)) hide)
-    )
-    (property "Datasheet" "" (at 95.25 100.33 0)
-      (effects (font (size 1.27 1.27)) hide)
-    )
-    (pin "1")
-    (instances
-      (project "dsoxlan"
-        (path "/071cacbe-efce-4cc8-8d6c-a55997c1e3c5"
-          (reference "#PWR02") (unit 1)
-        )
-      )
-    )
-  )
-  (symbol (lib_id "power:+3.3V") (at 95.25 107.95 0) (unit 1)
-    (in_bom yes) (on_board yes) (dnp no)
-    (property "Reference" "#PWR03" (at 95.25 111.76 0)
-      (effects (font (size 1.524 1.524)) hide)
-    )
-    (property "Value" "+3V3" (at 95.25 104.394 0)
-      (effects (font (size 1.524 1.524)))
-    )
-    (property "Footprint" "" (at 95.25 107.95 0)
-      (effects (font (size 1.27 1.27)) hide)
-    )
-    (property "Datasheet" "" (at 95.25 107.95 0)
-      (effects (font (size 1.27 1.27)) hide)
-    )
-    (pin "1")
-    (instances
-      (project "dsoxlan"
-        (path "/071cacbe-efce-4cc8-8d6c-a55997c1e3c5"
-          (reference "#PWR03") (unit 1)
         )
       )
@@
     )
   )
+  (symbol (lib_id "Device:R") (at 86.36 104.14 270) (unit 1)
+    (in_bom yes) (on_board yes) (dnp no)
+    (property "Reference" "R2" (at 86.36 106.172 90)
+      (effects (font (size 1.016 1.016)))
+    )
+    (property "Value" "470R" (at 86.3854 104.3178 90)
+      (effects (font (size 1.016 1.016)))
+    )
+    (property "Footprint" "Resistor_SMD:R_0805_2012Metric_Pad1.20x1.40mm_HandSolder" (at 86.36 102.362 90)
+      (effects (font (size 1.27 1.27)) hide)
+    )
+    (property "Datasheet" "~" (at 86.36 104.14 0)
+      (effects (font (size 1.27 1.27)) hide)
+    )
+    (pin "1")
+    (pin "2")
+    (instances
+      (project "dsoxlan"
+        (path "/071cacbe-efce-4cc8-8d6c-a55997c1e3c5"
+          (reference "R2") (unit 1)
+        )
+      )
+    )
+  )
   (symbol (lib_id "Mechanical:MountingHole") (at 83.82 139.7 0) (unit 1)
     (in_bom yes) (on_board yes) (dnp no) (fields_autoplaced)
@@
     )
   )
-  (symbol (lib_id "dsoxlan:WÜRTH-7499010121A") (at 67.31 88.9 0) (unit 1)
+  (symbol (lib_id "power:+3.3V") (at 95.25 96.52 0) (unit 1)
+    (in_bom yes) (on_board yes) (dnp no)
+    (property "Reference" "#PWR0103" (at 95.25 100.33 0)
+      (effects (font (size 1.524 1.524)) hide)
+    )
+    (property "Value" "+3V3" (at 95.25 92.964 0)
+      (effects (font (size 1.524 1.524)))
+    )
+    (property "Footprint" "" (at 95.25 96.52 0)
+      (effects (font (size 1.27 1.27)) hide)
+    )
+    (property "Datasheet" "" (at 95.25 96.52 0)
+      (effects (font (size 1.27 1.27)) hide)
+    )
+    (pin "1")
+    (instances
+      (project "dsoxlan"
+        (path "/071cacbe-efce-4cc8-8d6c-a55997c1e3c5"
+          (reference "#PWR0103") (unit 1)
+        )
+      )
+    )
+  )
+  (symbol (lib_id "dsoxlan:WÜRTH-7499011121A") (at 67.31 88.9 0) (unit 1)
     (in_bom yes) (on_board yes) (dnp no)
     (property "Reference" "P1" (at 73.66 67.31 0)
@@
       (effects (font (size 1.27 1.27)) (justify right))
     )
-    (property "Footprint" "DSOXLAN:WURTH-7499010121A" (at 53.34 92.71 90)
+    (property "Footprint" "DSOXLAN:7499011121A" (at 53.34 92.71 90)
       (effects (font (size 1.27 1.27)) hide)
     )
@@
         )
       )
+    )
+  )
+  (symbol (lib_id "Device:R") (at 86.36 96.52 270) (unit 1)
+    (in_bom yes) (on_board yes) (dnp no)
+    (property "Reference" "R1" (at 86.36 98.552 90)
+      (effects (font (size 1.016 1.016)))
+    )
+    (property "Value" "470R" (at 86.3854 96.6978 90)
+      (effects (font (size 1.016 1.016)))
+    )
+    (property "Footprint" "Resistor_SMD:R_0805_2012Metric_Pad1.20x1.40mm_HandSolder" (at 86.36 94.742 90)
+      (effects (font (size 1.27 1.27)) hide)
+    )
+    (property "Datasheet" "~" (at 86.36 96.52 0)
+      (effects (font (size 1.27 1.27)) hide)
+    )
+    (pin "1")
+    (pin "2")
+    (instances
+      (project "dsoxlan"
+        (path "/071cacbe-efce-4cc8-8d6c-a55997c1e3c5"
+          (reference "R1") (unit 1)
+        )
+      )
+    )
+  )
+  (symbol (lib_id "power:+3.3V") (at 95.25 104.14 0) (unit 1)
+    (in_bom yes) (on_board yes) (dnp no)
+    (property "Reference" "#PWR0102" (at 95.25 107.95 0)
+      (effects (font (size 1.524 1.524)) hide)
+    )
+    (property "Value" "+3V3" (at 95.25 100.584 0)
+      (effects (font (size 1.524 1.524)))
+    )
+    (property "Footprint" "" (at 95.25 104.14 0)
+      (effects (font (size 1.27 1.27)) hide)
+    )
+    (property "Datasheet" "" (at 95.25 104.14 0)
+      (effects (font (size 1.27 1.27)) hide)
+    )
+    (pin "1")
+    (instances
+      (project "dsoxlan"
+        (path "/071cacbe-efce-4cc8-8d6c-a55997c1e3c5"
+          (reference "#PWR0102") (unit 1)
+        )
+      )

Commit message: Add the housing parts to schematics
This allows to assign them correct reference designators, and
removes the DRC warnings about schematic parity mismatches.
Parts:
- added N1: Lid, DSOXLAN:Lid, symbol Mechanical:Housing
- added N2: Spacer1a, DSOXLAN:Spacer1a, symbol Mechanical:Housing
- added N3: Spacer2b, DSOXLAN:Spacer2b, symbol Mechanical:Housing
Changed lines of the file:
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@@
+    )
+  )
+  (symbol (lib_id "Mechanical:Housing") (at 43.18 152.4 0) (unit 1)
+    (in_bom yes) (on_board yes) (dnp no) (fields_autoplaced)
+    (property "Reference" "N2" (at 46.99 152.0738 0)
+      (effects (font (size 1.27 1.27)) (justify left))
+    )
+    (property "Value" "Spacer1a" (at 46.99 153.9948 0)
+      (effects (font (size 1.27 1.27)) (justify left))
+    )
+    (property "Footprint" "DSOXLAN:Spacer1a" (at 44.45 151.13 0)
+      (effects (font (size 1.27 1.27)) hide)
+    )
+    (property "Datasheet" "~" (at 44.45 151.13 0)
+      (effects (font (size 1.27 1.27)) hide)
+    )
+    (instances
+      (project "dsoxlan"
+        (path "/071cacbe-efce-4cc8-8d6c-a55997c1e3c5"
+          (reference "N2") (unit 1)
+        )
+      )
     )
   )
@@
         (path "/071cacbe-efce-4cc8-8d6c-a55997c1e3c5"
           (reference "#PWR0103") (unit 1)
+        )
+      )
+    )
+  )
+  (symbol (lib_id "Mechanical:Housing") (at 43.18 139.7 0) (unit 1)
+    (in_bom yes) (on_board yes) (dnp no) (fields_autoplaced)
+    (property "Reference" "N1" (at 46.99 139.3738 0)
+      (effects (font (size 1.27 1.27)) (justify left))
+    )
+    (property "Value" "Lid" (at 46.99 141.2948 0)
+      (effects (font (size 1.27 1.27)) (justify left))
+    )
+    (property "Footprint" "DSOXLAN:Lid" (at 44.45 138.43 0)
+      (effects (font (size 1.27 1.27)) hide)
+    )
+    (property "Datasheet" "~" (at 44.45 138.43 0)
+      (effects (font (size 1.27 1.27)) hide)
+    )
+    (instances
+      (project "dsoxlan"
+        (path "/071cacbe-efce-4cc8-8d6c-a55997c1e3c5"
+          (reference "N1") (unit 1)
         )
       )
@@
         )
       )
+    )
+  )
+  (symbol (lib_id "Mechanical:Housing") (at 43.18 166.37 0) (unit 1)
+    (in_bom yes) (on_board yes) (dnp no) (fields_autoplaced)
+    (property "Reference" "N3" (at 46.99 166.0438 0)
+      (effects (font (size 1.27 1.27)) (justify left))
+    )
+    (property "Value" "Spacer2b" (at 46.99 167.9648 0)
+      (effects (font (size 1.27 1.27)) (justify left))
+    )
+    (property "Footprint" "DSOXLAN:Spacer2b" (at 44.45 165.1 0)
+      (effects (font (size 1.27 1.27)) hide)
+    )
+    (property "Datasheet" "~" (at 44.45 165.1 0)
+      (effects (font (size 1.27 1.27)) hide)
+    )
+    (instances
+      (project "dsoxlan"
+        (path "/071cacbe-efce-4cc8-8d6c-a55997c1e3c5"
+          (reference "N3") (unit 1)
+        )
+      )
